File: CM4_GPIO.kicad_sch (KiCad schematic)
At the start: 28 parts, among them J1 Conn_01x03, J2 Conn_02x07_Odd_Even, J3 Conn_01x03, J7 Micro_SD_Card_Det, J8 THD-20-R, J9 THD-02-R, U1 TPD4EUSB30, U18 RT9742GGJ5, U2 TPD4EUSB30, U3 MagJack-A70-112-331N126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

Commit message: removed camera connector, ethernet ports and connections from CM4 Highspeed schematic and pcb. Re-arranged some traces and vias
Parts:
- removed C1: 100n, Capacitor_SMD:C_0402_1005Metric, symbol Device:C
- removed J9: THD-02-R, Connector_PinHeader_2.54mm:PinHeader_2x02_P2.54mm_Vertical, symbol Connector_Generic:Conn_02x02_Odd_Even
- removed R2, R3: 470R, Resistor_SMD:R_0402_1005Metric, symbol Device:R
- removed U1, U2: TPD4EUSB30, Package_SON:USON-10_2.5x1.0mm_P0.5mm, symbol CM4IO:TPD4EUSB30
- removed U3: MagJack-A70-112-331N126, CM4IO:TRJG0926HENL, symbol CM4IO:MagJack-A70-112-331N126
- C5: value 10u -> (none); footprint Capacitor_SMD:C_0805_2012Metric -> (none)
- D1: value LED Red -> (none); footprint LED_SMD:LED_0603_1608Metric -> (none)
- D2: value LED Green -> (none); footprint LED_SMD:LED_0603_1608Metric -> (none)
- J1, J3: value Conn_01x03 -> (none); footprint Connector_PinHeader_2.54mm:PinHeader_1x03_P2.54mm_Vertical -> (none)
- J2: value Conn_02x07_Odd_Even -> (none); footprint Connector_PinHeader_2.54mm:PinHeader_2x07_P2.54mm_Vertical -> (none)
- J7: value Micro_SD_Card_Det -> (none); footprint CM4IO:SDCARD_MOLEX_503398-1892 -> (none)
- J8: value THD-20-R -> (none); footprint Connector_PinHeader_2.54mm:PinHeader_2x20_P2.54mm_Vertical -> (none)
- Module1: value ComputeModule4 -> (none); footprint CM4IO:Raspberry-Pi-4-Compute-Module -> (none)
- R1, R10: value 1k -> (none); footprint Resistor_SMD:R_0402_1005Metric -> (none)
- R17, R18: value nf -> (none); footprint Resistor_SMD:R_0402_1005Metric -> (none)
- R29: value 12K 1% -> (none); footprint Resistor_SMD:R_0402_1005Metric -> (none)
- R4: value nf -> (none); footprint Resistor_SMD:R_0805_2012Metric_Pad1.15x1.40mm_HandSolder -> (none)
- R5: value 0R -> (none); footprint Resistor_SMD:R_0805_2012Metric_Pad1.15x1.40mm_HandSolder -> (none)
- TP3, TP5: value TestPoint -> (none); footprint TestPoint:TestPoint_Pad_2.0x2.0mm -> (none)
- U18: value RT9742GGJ5 -> (none); footprint Package_TO_SOT_SMD:SOT-23-5 -> (none)
- U5, U9: value 74LVC1G07SE-7 -> (none); footprint Package_TO_SOT_SMD:SOT-353_SC-70-5 -> (none)
Connections:
- net ETH_LEDG: no longer names the net of Module1.17 (Ethernet_nLED2(3.3v))
- net ETH_LEDY: no longer names the net of Module1.15 (Ethernet_nLED3(3.3v))
- net TRD0_N: no longer names the net of Module1.10 (Ethernet_Pair0_N)
- net TRD0_P: no longer names the net of Module1.12 (Ethernet_Pair0_P)
- net TRD1_N: no longer names the net of Module1.6 (Ethernet_Pair1_N)
- net TRD1_P: no longer names the net of Module1.4 (Ethernet_Pair1_P)
- net TRD2_N: no longer names the net of Module1.9 (Ethernet_Pair2_N)
- net TRD2_P: no longer names the net of Module1.11 (Ethernet_Pair2_P)
- net TRD3_N: no longer names the net of Module1.5 (Ethernet_Pair3_N)
- net TRD3_P: no longer names the net of Module1.3 (Ethernet_Pair3_P)
Other:
- note removed: "Ethernet"
- note removed: "Ethernet POE Protection"
- note removed: "POE Header"
